File: kicad/mb68k.kicad_pcb (KiCad board)
At the start: 2 copper layers, 38 parts, among them J1 Conn_01x06_Male, SW1 HW_RESET_SW, U1 NE555P, U10 74LS244, U11 68681, U2 74LS05, U3 68010P10, U4 GAL22V10, U5 SST39SF040, U6 AS6C4008-55PCN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

Commit message: Update footprint
Parts:
- C1: footprint Capacitor_THT:CP_Radial_D8.0mm_P5.00mm -> Capacitor_THT:CP_Radial_D10.0mm_P5.00mm
- C10, C11, C12, C13, C2, C3, C4, C5, C6, C7, C8, C9: footprint Capacitor_THT:CP_Radial_D8.0mm_P5.00mm -> Capacitor_THT:CP_Radial_D5.0mm_P2.50mm
- moved C8 226.4 mm to (129.5, 66.0)
- moved C6 136.7 mm to (162.6, 66.0)
- moved C7 2.54 mm to (132.1, 15.2)
- moved U5 2.54 mm to (154.9, 21.6)
- moved U8 2.54 mm to (121.9, 21.6)
