File: kicad/mb68k.kicad_pcb (KiCad board)
At the start: 4 copper layers, 130 parts, among them J1 Conn_01x01_Pin, J10 Free pin, J11 Free Pins, J12 Free pins, J13 Free pins, J14 Free pin, J15 Free pin, J16 Free pin, J17 Free pin, J18 Free pin, J19 Free pin, J2 Conn_01x06_Pin, J20 Spare resistors, J21 Power bar, J22 Spare resistors, J23 BUS Slot #1, J3 Conn_01x01_Pin, J4 Conn_01x01_Pin, J5 Conn_01x01_Pin, J6 PORTA serial, J7 PORTB serial, J8 DUART I/O, J9 Free pin, SW1 HW_RESET_SW, U1 74LS05, U10 GAL22V10, U11 AS6C4008-55PCN, U12 AS6C4008-55PCN, U13 74LS245, U14 74LS245, U15 68681, U16 GAL22V10, U17 GAL22V10, U18 74LS244, U19 74LS244, U2 NE555P, U20 74LS175, U3 74LS244, U4 GAL22V10, U5 SST39SF040, U6 SST39SF040, U7 68010P10, U8 74LS244, U9 74LS244, X1 SG-8002DB 10Mhz

Commit message: PCB to ATX size
Parts:
- removed C16, C17, C18: 100nF, Capacitor_THT:CP_Radial_D5.0mm_P2.50mm
- removed U13, U14: 74LS245, Package_DIP:DIP-20_W7.62mm_Socket
- removed U3, U8, U9: 74LS244, Package_DIP:DIP-20_W7.62mm_Socket
- added H1: MountingHole_Pad, MountingHole:MountingHole_4.3mm_M4_DIN965_Pad, F.Cu at (16.5, 237.5)
- added H10: MountingHole_Pad, MountingHole:MountingHole_4.3mm_M4_DIN965_Pad, F.Cu at (16.5, 10.2)
- added H2: MountingHole_Pad, MountingHole:MountingHole_4.3mm_M4_DIN965_Pad, F.Cu at (16.5, 165.1)
- added H3: MountingHole_Pad, MountingHole:MountingHole_4.3mm_M4_DIN965_Pad, F.Cu at (298.4, 165.1)
- added H4: MountingHole_Pad, MountingHole:MountingHole_4.3mm_M4_DIN965_Pad, F.Cu at (298.4, 33.0)
- added H5: MountingHole_Pad, MountingHole:MountingHole_4.3mm_M4_DIN965_Pad, F.Cu at (95.2, 10.2)
- added H6: MountingHole_Pad, MountingHole:MountingHole_4.3mm_M4_DIN965_Pad, F.Cu at (141.0, 237.5)
- added H7: MountingHole_Pad, MountingHole:MountingHole_4.3mm_M4_DIN965_Pad, F.Cu at (141.0, 165.1)
- added H8: MountingHole_Pad, MountingHole:MountingHole_4.3mm_M4_DIN965_Pad, F.Cu at (298.4, 237.5)
- added H9: MountingHole_Pad, MountingHole:MountingHole_4.3mm_M4_DIN965_Pad, F.Cu at (141.0, 10.2)
- added J24: BUS Slot 1, Connector_PinSocket_2.54mm:PinSocket_2x40_P2.54mm_Vertical, F.Cu at (32.0, 53.1)
- added J25: ATX-24, Connector_Molex:Molex_Mini-Fit_Jr_5566-24A_2x12_P4.20mm_Vertical, F.Cu at (232.1, 11.8)
- added LED3: GREEN PWR, LED_THT:LED_D5.0mm, F.Cu at (273.6, 222.8)
- added R41: R330, Resistor_THT:R_Axial_DIN0207_L6.3mm_D2.5mm_P10.16mm_Horizontal, F.Cu at (273.6, 203.2)
- added R42: R10 14W, Resistor_THT:R_Axial_Power_L50.0mm_W9.0mm_P60.96mm, F.Cu at (158.0, 14.2)
- added SW2: POWER ON, Button_Switch_SMD:SW_DIP_SPSTx01_Slide_6.7x4.1mm_W8.61mm_P2.54mm_LowProfile, F.Cu at (81.0, 221.0)
- C14: value 100nF -> 10uF
- J1, J3, J4, J5: value Conn_01x01_Pin -> Free pin
- J2: value Conn_01x06_Pin -> Free pins
- J23: value BUS Slot #1 -> BUS Slot 2
- U7: footprint Package_DIP:DIL64 -> Package_DIP:DIP-64_W25.4mm_Socket
- moved U11 589.5 mm to (202.4, 44.7)
- moved U12 589.5 mm to (225.3, 44.7)
- moved C8 506.0 mm to (211.4, 38.0), turned to 180 degrees
- moved U5 500.4 mm to (202.7, 104.4)
- moved U6 500.4 mm to (225.6, 104.4)
- moved J7 424.0 mm to (288.0, 211.1)
- moved J6 423.8 mm to (288.0, 131.6)
- moved J8 423.8 mm to (288.0, 154.4)
- moved C9 423.2 mm to (234.3, 38.0), turned to 180 degrees
- moved C28 412.7 mm to (247.9, 171.2)
- moved C11 407.8 mm to (234.5, 97.4), turned to 180 degrees
- moved 3.6864MHz1 394.8 mm to (278.4, 171.0)
- moved C19 394.8 mm to (275.9, 156.0)
- moved C20 394.8 mm to (275.9, 181.4)
- moved U15 394.8 mm to (255.5, 148.3)
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Connections:
- J21 pad 1: GND -> VCC
- J21 pad 10: VCC -> GND
- J21 pad 11: GND -> VCC
- J21 pad 12: VCC -> GND
- J21 pad 13: GND -> VCC
- J21 pad 14: VCC -> GND
- J21 pad 15: GND -> VCC
- J21 pad 16: VCC -> GND
- J21 pad 17: GND -> VCC
- J21 pad 18: VCC -> GND
- J21 pad 19: GND -> VCC
- J21 pad 2: VCC -> GND
- J21 pad 20: VCC -> GND
- J21 pad 21: GND -> VCC
- J21 pad 22: VCC -> GND
- J21 pad 3: GND -> VCC
- J21 pad 4: VCC -> GND
- J21 pad 5: GND -> VCC
- J21 pad 6: VCC -> GND
- J21 pad 7: GND -> VCC
- J21 pad 8: VCC -> GND
- J21 pad 9: GND -> VCC
- J23 pad 10: A_BUF9 -> unconnected-(J23-Pin_10-Pad10)
- J23 pad 11: A_BUF10 -> A19
- J23 pad 12: A_BUF11 -> ~{DTACK}
- J23 pad 13: A_BUF12 -> A18
- J23 pad 14: A_BUF13 -> unconnected-(J23-Pin_14-Pad14)
- J23 pad 15: A_BUF14 -> A17
- J23 pad 16: A_BUF15 -> unconnected-(J23-Pin_16-Pad16)
- J23 pad 17: A_BUF16 -> A16
- J23 pad 18: A_BUF17 -> unconnected-(J23-Pin_18-Pad18)
- J23 pad 19: A_BUF18 -> A15
- J23 pad 2: A_BUF1 -> GND
- J23 pad 20: A_BUF19 -> _R/~{W}
- J23 pad 21: A_BUF20 -> A14
- J23 pad 22: A_BUF21 -> ~{_LDS}
- J23 pad 23: A_BUF22 -> A13
- J23 pad 24: A_BUF23 -> ~{_UDS}
- J23 pad 25: VCC -> A12
- J23 pad 26: ~{IACK1} -> ~{_AS}
- J23 pad 27: ~{IACK2} -> A11
- J23 pad 28: ~{IACK3} -> unconnected-(J23-Pin_28-Pad28)
- J23 pad 29: ~{IACK4} -> A10
- J23 pad 3: A_BUF2 -> A23
- J23 pad 30: ~{IACK5} -> unconnected-(J23-Pin_30-Pad30)
- J23 pad 31: ~{IACK6} -> A9
- J23 pad 32: ~{IACK7} -> ~{IRQ1}
- J23 pad 33: unconnected-(J23-Pin_33-Pad33) -> A8
- J23 pad 34: unconnected-(J23-Pin_34-Pad34) -> ~{IRQ2}
- J23 pad 35: unconnected-(J23-Pin_35-Pad35) -> A7
- J23 pad 36: unconnected-(J23-Pin_36-Pad36) -> ~{IRQ3}
- J23 pad 37: unconnected-(J23-Pin_37-Pad37) -> A6
- J23 pad 38: unconnected-(J23-Pin_38-Pad38) -> ~{IRQ4}
- J23 pad 39: unconnected-(J23-Pin_39-Pad39) -> A5
- J23 pad 4: A_BUF3 -> CLK
- J23 pad 40: unconnected-(J23-Pin_40-Pad40) -> ~{IRQ5}
- J23 pad 41: unconnected-(J23-Pin_41-Pad41) -> A4
- J23 pad 42: D_BUF15 -> ~{IRQ6}
- J23 pad 43: D_BUF14 -> A3
- J23 pad 44: D_BUF13 -> ~{IRQ7}
- J23 pad 45: D_BUF12 -> A2
- J23 pad 46: D_BUF11 -> GND
- J23 pad 47: D_BUF10 -> A1
- J23 pad 48: D_BUF9 -> D15
- J23 pad 49: D_BUF8 -> VCC
- J23 pad 5: A_BUF4 -> A22
- J23 pad 50: D_BUF7 -> D14
- J23 pad 51: D_BUF6 -> ~{IACK1}
- J23 pad 52: D_BUF5 -> D13
- J23 pad 53: D_BUF4 -> ~{IACK2}
- J23 pad 54: D_BUF3 -> D12
- J23 pad 55: D_BUF2 -> ~{IACK3}
- J23 pad 56: D_BUF1 -> D11
- J23 pad 57: D_BUF0 -> ~{IACK4}
- J23 pad 58: GND -> D10
- J23 pad 59: ~{IRQ7} -> ~{IACK5}
- J23 pad 6: A_BUF5 -> unconnected-(J23-Pin_6-Pad6)
- J23 pad 60: ~{IRQ6} -> D9
- J23 pad 61: ~{IRQ5} -> ~{IACK6}
- J23 pad 62: ~{IRQ4} -> D8
- J23 pad 63: ~{IRQ3} -> ~{IACK7}
- J23 pad 64: ~{IRQ2} -> D7
- J23 pad 65: ~{IRQ1} -> unconnected-(J23-Pin_65-Pad65)
- J23 pad 66: unconnected-(J23-Pin_66-Pad66) -> D6
- J23 pad 68: ~{_AS} -> D5
- J23 pad 69: ~{_UDS} -> unconnected-(J23-Pin_69-Pad69)
- J23 pad 7: A_BUF6 -> A21
- J23 pad 70: ~{_LDS} -> D4
- J23 pad 71: _R/~{W} -> unconnected-(J23-Pin_71-Pad71)
- J23 pad 72: unconnected-(J23-Pin_72-Pad72) -> D3
- J23 pad 74: unconnected-(J23-Pin_74-Pad74) -> D2
- J23 pad 75: ~{DTACK} -> unconnected-(J23-Pin_75-Pad75)
- J23 pad 76: unconnected-(J23-Pin_76-Pad76) -> D1
- J23 pad 78: unconnected-(J23-Pin_78-Pad78) -> D0
- J23 pad 79: CLK -> unconnected-(J23-Pin_79-Pad79)
- J23 pad 8: A_BUF7 -> unconnected-(J23-Pin_8-Pad8)
- J23 pad 80: GND -> unconnected-(J23-Pin_80-Pad80)
- J23 pad 9: A_BUF8 -> A20
- U11 pad 1: A_BUF19 -> A19
- U11 pad 10: A_BUF3 -> A3
- U11 pad 11: A_BUF2 -> A2
- U11 pad 12: A_BUF1 -> A1
- U11 pad 13: D_BUF0 -> D0
- U11 pad 14: D_BUF1 -> D1
- U11 pad 15: D_BUF2 -> D2
- U11 pad 17: D_BUF3 -> D3
- U11 pad 18: D_BUF4 -> D4
- U11 pad 19: D_BUF5 -> D5
- U11 pad 2: A_BUF17 -> A17
- U11 pad 20: D_BUF6 -> D6
- U11 pad 21: D_BUF7 -> D7
- U11 pad 23: A_BUF11 -> A11
- U11 pad 25: A_BUF12 -> A12
- U11 pad 26: A_BUF10 -> A10
- U11 pad 27: A_BUF9 -> A9
- U11 pad 28: A_BUF14 -> A14
- U11 pad 3: A_BUF15 -> A15
- U11 pad 30: A_BUF18 -> A18
- U11 pad 31: A_BUF16 -> A16
- U11 pad 4: A_BUF13 -> A13
- U11 pad 5: A_BUF8 -> A8
- U11 pad 6: A_BUF7 -> A7
- U11 pad 7: A_BUF6 -> A6
- U11 pad 8: A_BUF5 -> A5
- U11 pad 9: A_BUF4 -> A4
- U12 pad 1: A_BUF19 -> A19
- U12 pad 10: A_BUF3 -> A3
- U12 pad 11: A_BUF2 -> A2
- U12 pad 12: A_BUF1 -> A1
- U12 pad 13: D_BUF8 -> D8
- U12 pad 14: D_BUF9 -> D9
- U12 pad 15: D_BUF10 -> D10
- U12 pad 17: D_BUF11 -> D11
- U12 pad 18: D_BUF12 -> D12
- U12 pad 19: D_BUF13 -> D13
- U12 pad 2: A_BUF17 -> A17
- U12 pad 20: D_BUF14 -> D14
- U12 pad 21: D_BUF15 -> D15
- U12 pad 23: A_BUF11 -> A11
- U12 pad 25: A_BUF12 -> A12
- U12 pad 26: A_BUF10 -> A10
- U12 pad 27: A_BUF9 -> A9
- U12 pad 28: A_BUF14 -> A14
- U12 pad 3: A_BUF15 -> A15
- U12 pad 30: A_BUF18 -> A18
- U12 pad 31: A_BUF16 -> A16
- U12 pad 4: A_BUF13 -> A13
- U12 pad 5: A_BUF8 -> A8
- U12 pad 6: A_BUF7 -> A7
- U12 pad 7: A_BUF6 -> A6
- U12 pad 8: A_BUF5 -> A5
- U12 pad 9: A_BUF4 -> A4
- U15 pad 1: A_BUF1 -> A1
- U15 pad 16: D_BUF1 -> D1
- U15 pad 17: D_BUF3 -> D3
- U15 pad 18: D_BUF5 -> D5
- U15 pad 19: D_BUF7 -> D7
- U15 pad 22: D_BUF6 -> D6
- U15 pad 23: D_BUF4 -> D4
- U15 pad 24: D_BUF2 -> D2
- U15 pad 25: D_BUF0 -> D0
- U15 pad 3: A_BUF2 -> A2
- U15 pad 5: A_BUF3 -> A3
- U15 pad 6: A_BUF4 -> A4
- U5 pad 1: A_BUF19 -> A19
- U5 pad 10: A_BUF3 -> A3
- U5 pad 11: A_BUF2 -> A2
- U5 pad 12: A_BUF1 -> A1
- U5 pad 13: D_BUF0 -> D0
- U5 pad 14: D_BUF1 -> D1
- U5 pad 15: D_BUF2 -> D2
- U5 pad 17: D_BUF3 -> D3
- U5 pad 18: D_BUF4 -> D4
- U5 pad 19: D_BUF5 -> D5
- U5 pad 2: A_BUF17 -> A17
- U5 pad 20: D_BUF6 -> D6
- U5 pad 21: D_BUF7 -> D7
- U5 pad 23: A_BUF11 -> A11
- U5 pad 25: A_BUF12 -> A12
- U5 pad 26: A_BUF10 -> A10
- U5 pad 27: A_BUF9 -> A9
- U5 pad 28: A_BUF14 -> A14
- U5 pad 29: A_BUF15 -> A15
- U5 pad 3: A_BUF16 -> A16
- U5 pad 30: A_BUF18 -> A18
- U5 pad 4: A_BUF13 -> A13
- U5 pad 5: A_BUF8 -> A8
- U5 pad 6: A_BUF7 -> A7
- U5 pad 7: A_BUF6 -> A6
- U5 pad 8: A_BUF5 -> A5
- U5 pad 9: A_BUF4 -> A4
- U6 pad 1: A_BUF19 -> A19
- U6 pad 10: A_BUF3 -> A3
- U6 pad 11: A_BUF2 -> A2
- U6 pad 12: A_BUF1 -> A1
- U6 pad 13: D_BUF8 -> D8
- U6 pad 14: D_BUF9 -> D9
- U6 pad 15: D_BUF10 -> D10
- U6 pad 17: D_BUF11 -> D11
- U6 pad 18: D_BUF12 -> D12
- U6 pad 19: D_BUF13 -> D13
- U6 pad 2: A_BUF17 -> A17
- U6 pad 20: D_BUF14 -> D14
- U6 pad 21: D_BUF15 -> D15
- U6 pad 23: A_BUF11 -> A11
- U6 pad 25: A_BUF12 -> A12
- U6 pad 26: A_BUF10 -> A10
- U6 pad 27: A_BUF9 -> A9
- U6 pad 28: A_BUF14 -> A14
- U6 pad 29: A_BUF15 -> A15
- U6 pad 3: A_BUF16 -> A16
- U6 pad 30: A_BUF18 -> A18
- U6 pad 4: A_BUF13 -> A13
- U6 pad 5: A_BUF8 -> A8
- U6 pad 6: A_BUF7 -> A7
- U6 pad 7: A_BUF6 -> A6
- U6 pad 8: A_BUF5 -> A5
- U6 pad 9: A_BUF4 -> A4
Other:
- board outline added: 305 x 244 mm

Commit message: saving state
Parts:
- added C16: 100uF, Capacitor_THT:CP_Radial_D5.0mm_P2.50mm, F.Cu at (262.6, 31.3)
- added C17: 470uF, Capacitor_THT:CP_Radial_D5.0mm_P2.50mm, F.Cu at (269.2, 31.3)
- added J26: External Power, Connector_PinHeader_2.54mm:PinHeader_1x02_P2.54mm_Vertical, F.Cu at (275.3, 31.2)
- added JP1: BASE LOAD, Connector_PinHeader_2.54mm:PinHeader_2x01_P2.54mm_Vertical, F.Cu at (220.5, 16.5)
- C1, C10, C11, C12, C13, C19, C20, C21, C22, C23, C24, C25, C27, C28, C3, C4, C8, C9: footprint Capacitor_THT:CP_Radial_D5.0mm_P2.50mm -> Capacitor_THT:C_Disc_D5.0mm_W2.5mm_P2.50mm
- J21: footprint Connector_PinSocket_2.54mm:PinSocket_2x11_P2.54mm_Vertical -> Connector_PinSocket_2.54mm:PinSocket_2x10_P2.54mm_Vertical
- moved J6 93.1 mm to (292.6, 224.6), turned to -90 degrees
- moved C28 29.9 mm to (261.9, 144.8)
- moved C25 18.5 mm to (13.4, 34.8)
- moved C26 18.5 mm to (13.5, 44.2)
- moved J24 18.5 mm to (13.5, 52.8)
- moved C8 14.4 mm to (211.8, 52.3)
- moved C9 14.4 mm to (234.1, 52.3)
- moved U11 11.7 mm to (202.7, 56.4)
- moved U12 11.7 mm to (225.6, 56.4)
- moved R10 7.11 mm to (110.5, 157.5)
- moved R12 7.11 mm to (124.2, 157.5)
- moved R11 7.11 mm to (117.3, 157.5)
- moved R13 6.10 mm to (131.8, 157.5)
- moved J18 5.62 mm to (160.0, 180.3)
- moved J19 5.33 mm to (157.5, 196.1)
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Connections:
- J23 pad 18: unconnected-(J23-Pin_18-Pad18) -> ~{EXTSEL}
- J23 pad 32: ~{IRQ1} -> D4
- J23 pad 34: ~{IRQ2} -> D3
- J23 pad 36: ~{IRQ3} -> D2
- J23 pad 38: ~{IRQ4} -> D1
- J23 pad 40: ~{IRQ5} -> D0
- J23 pad 42: ~{IRQ6} -> GND
- J23 pad 46: GND -> ~{IRQ6}
- J23 pad 48: D15 -> ~{IRQ5}
- J23 pad 50: D14 -> ~{IRQ4}
- J23 pad 51: ~{IACK1} -> ~{IACK7}
- J23 pad 52: D13 -> ~{IRQ3}
- J23 pad 53: ~{IACK2} -> ~{IACK6}
- J23 pad 54: D12 -> ~{IRQ2}
- J23 pad 55: ~{IACK3} -> ~{IACK5}
- J23 pad 56: D11 -> ~{IRQ1}
- J23 pad 58: D10 -> D5
- J23 pad 59: ~{IACK5} -> ~{IACK3}
- J23 pad 60: D9 -> D6
- J23 pad 61: ~{IACK6} -> ~{IACK2}
- J23 pad 62: D8 -> D7
- J23 pad 63: ~{IACK7} -> ~{IACK1}
- J23 pad 64: D7 -> D8
- J23 pad 66: D6 -> D9
- J23 pad 68: D5 -> D10
- J23 pad 70: D4 -> D11
- J23 pad 72: D3 -> D12
- J23 pad 74: D2 -> D13
- J23 pad 76: D1 -> D14
- J23 pad 78: D0 -> D15
- J24 pad 18: unconnected-(J24-Pin_18-Pad18) -> ~{EXTSEL}
- J24 pad 32: ~{IRQ1} -> D4
- J24 pad 34: ~{IRQ2} -> D3
- J24 pad 36: ~{IRQ3} -> D2
- J24 pad 38: ~{IRQ4} -> D1
- J24 pad 40: ~{IRQ5} -> D0
- J24 pad 42: ~{IRQ6} -> GND
- J24 pad 46: GND -> ~{IRQ6}
- J24 pad 48: D15 -> ~{IRQ5}
- J24 pad 50: D14 -> ~{IRQ4}
- J24 pad 51: ~{IACK1} -> ~{IACK7}
- J24 pad 52: D13 -> ~{IRQ3}
- J24 pad 53: ~{IACK2} -> ~{IACK6}
- J24 pad 54: D12 -> ~{IRQ2}
- J24 pad 55: ~{IACK3} -> ~{IACK5}
- J24 pad 56: D11 -> ~{IRQ1}
- J24 pad 58: D10 -> D5
- J24 pad 59: ~{IACK5} -> ~{IACK3}
- J24 pad 60: D9 -> D6
- J24 pad 61: ~{IACK6} -> ~{IACK2}
- J24 pad 62: D8 -> D7
- J24 pad 63: ~{IACK7} -> ~{IACK1}
- J24 pad 64: D7 -> D8
- J24 pad 66: D6 -> D9
- J24 pad 68: D5 -> D10
- J24 pad 70: D4 -> D11
- J24 pad 72: D3 -> D12
- J24 pad 74: D2 -> D13
- J24 pad 76: D1 -> D14
- J24 pad 78: D0 -> D15
- R42 pad 2: GND -> Net-(JP1-B)
- U10 pad 22: unconnected-(U10-I/O-Pad22) -> ~{EXTSEL}
Other:
- board text added: "+5v"
- board text added: "Even RAM0"
- board text added: "Even ROM"
- board text added: "GND"
- board text added: "Odd RAM0"
- board text added: "Odd ROM"
- board text added: "RX"
- board text added: "TX"
