File: kicad/Reset.kicad_sch (KiCad schematic)
At the start: 20 parts, among them J1 Power, J2 Halt_Reset, U1 NE555P, U2 74LS05, X1 SG-8002DB 10Mhz

Commit message: started with pcb
Parts:
- removed J1: Power, Connector_PinHeader_2.54mm:PinHeader_1x02_P2.54mm_Vertical, symbol Connector_Generic:Conn_02x01
- removed J2: Halt_Reset, Connector_PinHeader_2.54mm:PinHeader_1x02_P2.54mm_Vertical, symbol Connector_Generic:Conn_01x02
- removed S1: 10-XX, matsb:B3F-10XX, symbol rosco_m68k-eagle-import:10-XX
- added SW1: HW_RESET_SW, Button_Switch_SMD:SW_MEC_5GSH9, symbol Switch:SW_MEC_5E
- C2, C3, C4, C5: footprint Capacitor_THT:C_Disc_D4.3mm_W1.9mm_P5.00mm -> Capacitor_THT:CP_Radial_D8.0mm_P5.00mm
- X1: footprint Oscillator:Oscillator_SeikoEpson_SG-8002DB -> Oscillator:Oscillator_DIP-14
Connections:
- net at R2.1: now also SW1.1
- net at C1.1, R1.2, U1.2 (TR)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: now also SW1.3 (K)
- no-connect marks 3 -> 4
Other:
- title: Mats Brorson 68010 SBC -> Mats Brorson 68010 SBC Clock circuit
- moved on the sheet: R2

Commit message: Update footprint
Parts:
- C1: footprint Capacitor_THT:CP_Radial_D8.0mm_P5.00mm -> Capacitor_THT:CP_Radial_D10.0mm_P5.00mm
- C2, C3, C4, C5: footprint Capacitor_THT:CP_Radial_D8.0mm_P5.00mm -> Capacitor_THT:CP_Radial_D5.0mm_P2.50mm
Changed lines of the file:
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@@
       (effects (font (size 1.27 1.27)) (justify left))
     )
-    (property "Footprint" "Capacitor_THT:CP_Radial_D8.0mm_P5.00mm" (id 2) (at 105.1052 120.65 0)
+    (property "Footprint" "Capacitor_THT:CP_Radial_D5.0mm_P2.50mm" (id 2) (at 105.1052 120.65 0)
       (effects (font (size 1.27 1.27)) hide)
     )
@@
       (effects (font (size 1.27 1.27)) (justify left))
     )
-    (property "Footprint" "Capacitor_THT:CP_Radial_D8.0mm_P5.00mm" (id 2) (at 204.1652 140.97 0)
+    (property "Footprint" "Capacitor_THT:CP_Radial_D5.0mm_P2.50mm" (id 2) (at 204.1652 140.97 0)
       (effects (font (size 1.27 1.27)) hide)
     )
@@
       (effects (font (size 1.27 1.27)) (justify left))
     )
-    (property "Footprint" "Capacitor_THT:CP_Radial_D8.0mm_P5.00mm" (id 2) (at 26.3652 97.79 0)
+    (property "Footprint" "Capacitor_THT:CP_Radial_D10.0mm_P5.00mm" (id 2) (at 26.3652 97.79 0)
       (effects (font (size 1.27 1.27)) hide)
     )
@@
       (effects (font (size 1.27 1.27)) (justify left))
     )
-    (property "Footprint" "Capacitor_THT:CP_Radial_D8.0mm_P5.00mm" (id 2) (at 265.1252 140.97 0)
+    (property "Footprint" "Capacitor_THT:CP_Radial_D5.0mm_P2.50mm" (id 2) (at 265.1252 140.97 0)
       (effects (font (size 1.27 1.27)) hide)
     )
@@
       (effects (font (size 1.27 1.27)) (justify left))
     )
-    (property "Footprint" "Capacitor_THT:CP_Radial_D8.0mm_P5.00mm" (id 2) (at 44.1452 67.31 0)
-      (effects (font (size 1.27 1.27)) hide)
-    )
+    (property "Footprint" "Capacitor_THT:CP_Radial_D5.0mm_P2.50mm" (id 2) (at 44.1452 67.31 0)
+      (effects (font (size 1.27 1.27)) hide)
+    )
