File: kicad/Reset.kicad_sch (KiCad schematic)
At the start: 18 parts, among them SW1 HW_RESET_SW, U1 NE555P, U2 74LS05, X1 SG-8002DB 10Mhz

Commit message: New decoding and GALs
Parts:
- added unit 5 of U2
- added unit 6 of U2
- added unit 4 of U2
Connections:
- net /HALT renamed ~{HALT}
- net /RESET renamed ~{RESET}
- no-connect marks 4 -> 9
Other:
- moved on the sheet: C3, U2G

Commit message: added footprints
Parts:
- C2: renamed from C1; footprint Capacitor_THT:CP_Radial_D10.0mm_P5.00mm -> Capacitor_THT:CP_Radial_D5.0mm_P2.50mm
- U1: renamed from U2; footprint (none) -> Package_DIP:DIP-14_W7.62mm
- renumbered C2 to C1, R3 to R1, R4 to R2, R5 to R3, R6 to R4, R1 to R5, R7 to R6, R2 to R7, U2 to U1, U1 to U2

Commit message: PCB to ATX size
Changed lines of the file:
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@@
-    (stroke (width 0) (type default))
-  )
-  (wire (pts (xy 275.59 53.34) (xy 275.59 67.31))
     (stroke (width 0) (type default))
   )
@@
   )
   (wire (pts (xy 170.18 34.29) (xy 170.18 44.45))
-    (stroke (width 0) (type default))
-  )
-  (wire (pts (xy 257.81 53.34) (xy 257.81 67.31))
     (stroke (width 0) (type default))
   )
@@
     )
   )
-  (symbol (lib_id "power:VCC") (at 257.81 53.34 0) (unit 1)
-    (in_bom yes) (on_board yes) (dnp no)
-    (property "Reference" "#PWR02" (at 257.81 57.15 0)
-      (effects (font (size 1.27 1.27)) hide)
-    )
-    (property "Value" "VCC" (at 257.81 48.26 0)
-      (effects (font (size 1.27 1.27)))
-    )
-    (property "Footprint" "" (at 257.81 53.34 0)
-      (effects (font (size 1.27 1.27)) hide)
-    )
-    (property "Datasheet" "" (at 257.81 53.34 0)
-      (effects (font (size 1.27 1.27)) hide)
-    )
-    (pin "1")
-    (instances
-      (project "mb68k"
-        (path "/e63e39d7-6ac0-4ffd-8aa3-1841a4541b55/60b3e0cc-7d6f-4628-b20d-5a9d7b2fa5fa"
-          (reference "#PWR02") (unit 1)
-        )
-      )
-    )
-  )
   (symbol (lib_id "Device:R") (at 130.81 48.26 0) (unit 1)
     (in_bom yes) (on_board yes) (dnp no) (fields_autoplaced)
@@
         (path "/e63e39d7-6ac0-4ffd-8aa3-1841a4541b55/60b3e0cc-7d6f-4628-b20d-5a9d7b2fa5fa"
           (reference "R1") (unit 1)
-        )
-      )
-    )
-  )
-  (symbol (lib_id "power:PWR_FLAG") (at 257.81 67.31 180) (unit 1)
-    (in_bom yes) (on_board yes) (dnp no)
-    (property "Reference" "#FLG02" (at 257.81 69.215 0)
-      (effects (font (size 1.27 1.27)) hide)
-    )
-    (property "Value" "PWR_FLAG" (at 252.73 72.39 0)
-      (effects (font (size 1.27 1.27)) (justify right))
-    )
-    (property "Footprint" "" (at 257.81 67.31 0)
-      (effects (font (size 1.27 1.27)) hide)
-    )
-    (property "Datasheet" "~" (at 257.81 67.31 0)
-      (effects (font (size 1.27 1.27)) hide)
-    )
-    (pin "1")
-    (instances
-      (project "mb68k"
-        (path "/e63e39d7-6ac0-4ffd-8aa3-1841a4541b55/60b3e0cc-7d6f-4628-b20d-5a9d7b2fa5fa"
-          (reference "#FLG02") (unit 1)
         )
       )
@@
     )
   )
-  (symbol (lib_id "power:PWR_FLAG") (at 275.59 53.34 0) (unit 1)
-    (in_bom yes) (on_board yes) (dnp no) (fields_autoplaced)
-    (property "Reference" "#FLG01" (at 275.59 51.435 0)
-      (effects (font (size 1.27 1.27)) hide)
-    )
-    (property "Value" "PWR_FLAG" (at 275.59 48.26 0)
-      (effects (font (size 1.27 1.27)))
-    )
-    (property "Footprint" "" (at 275.59 53.34 0)
-      (effects (font (size 1.27 1.27)) hide)
-    )
-    (property "Datasheet" "~" (at 275.59 53.34 0)
-      (effects (font (size 1.27 1.27)) hide)
-    )
-    (pin "1")
-    (instances
-      (project "mb68k"
-        (path "/e63e39d7-6ac0-4ffd-8aa3-1841a4541b55/60b3e0cc-7d6f-4628-b20d-5a9d7b2fa5fa"
-          (reference "#FLG01") (unit 1)
-        )
-      )
-    )
-  )
   (symbol (lib_id "Device:R") (at 170.18 48.26 0) (unit 1)
     (in_bom yes) (on_board yes) (dnp no) (fields_autoplaced)
@@
         )
       )
-    )
-  )
-  (symbol (lib_id "power:GND") (at 275.59 67.31 0) (unit 1)
-    (in_bom yes) (on_board yes) (dnp no)
-    (property "Reference" "#PWR03" (at 275.59 73.66 0)
-      (effects (font (size 1.27 1.27)) hide)
-    )
-    (property "Value" "GND" (at 276.86 72.39 0)
-      (effects (font (size 1.27 1.27)) (justify right))
-    )
-    (property "Footprint" "" (at 275.59 67.31 0)
-      (effects (font (size 1.27 1.27)) hide)
-    )
-    (property "Datasheet" "" (at 275.59 67.31 0)
-      (effects (font (size 1.27 1.27)) hide)
-    )
-    (pin "1")
-    (instances
-      (project "mb68k"
-        (path "/e63e39d7-6ac0-4ffd-8aa3-1841a4541b55/60b3e0cc-7d6f-4628-b20d-5a9d7b2fa5fa"
-          (reference "#PWR03") (unit 1)
-        )
-      )

Commit message: saving state
Parts:
- C1, C3, C4: footprint Capacitor_THT:CP_Radial_D5.0mm_P2.50mm -> Capacitor_THT:C_Disc_D5.0mm_W2.5mm_P2.50mm
Changed lines of the file:
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@@
       (effects (font (size 1.27 1.27)) (justify left))
     )
-    (property "Footprint" "Capacitor_THT:CP_Radial_D5.0mm_P2.50mm" (at 105.1052 123.19 0)
+    (property "Footprint" "Capacitor_THT:C_Disc_D5.0mm_W2.5mm_P2.50mm" (at 105.1052 123.19 0)
       (effects (font (size 1.27 1.27)) hide)
     )
@@
       (effects (font (size 1.27 1.27)) (justify left))
     )
-    (property "Footprint" "Capacitor_THT:CP_Radial_D5.0mm_P2.50mm" (at 204.1652 140.97 0)
+    (property "Footprint" "Capacitor_THT:C_Disc_D5.0mm_W2.5mm_P2.50mm" (at 204.1652 140.97 0)
       (effects (font (size 1.27 1.27)) hide)
     )
@@
       (effects (font (size 1.27 1.27)) (justify left))
     )
-    (property "Footprint" "Capacitor_THT:CP_Radial_D5.0mm_P2.50mm" (at 44.1452 67.31 0)
-      (effects (font (size 1.27 1.27)) hide)
-    )
+    (property "Footprint" "Capacitor_THT:C_Disc_D5.0mm_W2.5mm_P2.50mm" (at 44.1452 67.31 0)
+      (effects (font (size 1.27 1.27)) hide)
+    )

Commit message: got irq to work
Parts:
- removed SW1: HW_RESET_SW, Button_Switch_SMD:SW_MEC_5GSH9, symbol Switch:SW_MEC_5E
- added SW1: Reset, Button_Switch_THT:SW_PUSH_6mm, symbol Switch:SW_DIP_x01
Connections:
- net at R7.1: now also SW1.2
- net at C2.1, R5.2, U2.2 (TR)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: now also SW1.1
- no-connect marks 9 -> 7
Changed lines of the file:
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@@
   (no_connect (at 147.32 139.7))
   (no_connect (at 132.08 154.94))
-  (no_connect (at 38.1 140.97))
   (no_connect (at 132.08 139.7))
   (no_connect (at 72.39 81.28))
-  (no_connect (at 48.26 138.43))
   (wire (pts (xy 156.21 64.77) (xy 156.21 76.2))
     (stroke (width 0) (type default))
@@
     (stroke (width 0) (type default))
   )
-  (wire (pts (xy 38.1 138.43) (xy 25.4 138.43))
-    (stroke (width 0) (type default))
-  )
   (wire (pts (xy 218.44 137.16) (xy 213.36 137.16))
     (stroke (width 0) (type default))
@@
     (stroke (width 0) (type default))
   )
+  (wire (pts (xy 25.4 140.97) (xy 33.02 140.97))
+    (stroke (width 0) (type default))
+  )
   (wire (pts (xy 35.56 34.29) (xy 43.18 34.29))
     (stroke (width 0) (type default))
@@
     (stroke (width 0) (type default))
   )
-  (wire (pts (xy 25.4 138.43) (xy 25.4 114.3))
+  (wire (pts (xy 25.4 114.3) (xy 25.4 140.97))
     (stroke (width 0) (type default))
   )
@@
         (path "/e63e39d7-6ac0-4ffd-8aa3-1841a4541b55/60b3e0cc-7d6f-4628-b20d-5a9d7b2fa5fa"
           (reference "X1") (unit 1)
-        )
-      )
-    )
-  )
-  (symbol (lib_id "Switch:SW_MEC_5E") (at 43.18 138.43 180) (unit 1)
-    (in_bom yes) (on_board yes) (dnp no)
-    (property "Reference" "SW1" (at 43.18 148.59 0)
-      (effects (font (size 1.27 1.27)))
-    )
-    (property "Value" "HW_RESET_SW" (at 43.18 146.05 0)
-      (effects (font (size 1.27 1.27)))
-    )
-    (property "Footprint" "Button_Switch_SMD:SW_MEC_5GSH9" (at 43.18 146.05 0)
-      (effects (font (size 1.27 1.27)) hide)
-    )
-    (property "Datasheet" "http://www.apem.com/int/index.php?controller=attachment&id_attachment=1371" (at 43.18 146.05 0)
-      (effects (font (size 1.27 1.27)) hide)
-    )
-    (pin "1")
-    (pin "2")
-    (pin "3")
-    (pin "4")
-    (instances
-      (project "mb68k"
-        (path "/e63e39d7-6ac0-4ffd-8aa3-1841a4541b55/60b3e0cc-7d6f-4628-b20d-5a9d7b2fa5fa"
-          (reference "SW1") (unit 1)
         )
       )
@@
         )
       )
+    )
+  )
+  (symbol (lib_id "Switch:SW_DIP_x01") (at 40.64 140.97 0) (unit 1)
+    (in_bom yes) (on_board yes) (dnp no) (fields_autoplaced)
+    (property "Reference" "SW1" (at 40.64 133.35 0)
+      (effects (font (size 1.27 1.27)))
+    )
+    (property "Value" "Reset" (at 40.64 135.89 0)
+      (effects (font (size 1.27 1.27)))
+    )
+    (property "Footprint" "Button_Switch_THT:SW_PUSH_6mm" (at 40.64 140.97 0)
+      (effects (font (size 1.27 1.27)) hide)
+    )
+    (property "Datasheet" "~" (at 40.64 140.97 0)
+      (effects (font (size 1.27 1.27)) hide)
+    )
+    (pin "1")
+    (pin "2")
+    (instances
+      (project "mb68k"
+        (path "/e63e39d7-6ac0-4ffd-8aa3-1841a4541b55/60b3e0cc-7d6f-4628-b20d-5a9d7b2fa5fa"
+          (reference "SW1") (unit 1)
+        )
+      )
