File: kicad/_autosave-mb68k.kicad_pcb (KiCad board)
At the start: 4 copper layers, 130 parts, among them J1 Conn_01x01_Pin, J10 Free pin, J11 Free Pins, J12 Free pins, J13 Free pins, J14 Free pin, J15 Free pin, J16 Free pin, J17 Free pin, J18 Free pin, J19 Free pin, J2 Conn_01x06_Pin, J20 Spare resistors, J21 Power bar, J22 Spare resistors, J23 BUS Slot #1, J3 Conn_01x01_Pin, J4 Conn_01x01_Pin, J5 Conn_01x01_Pin, J6 PORTA serial, J7 PORTB serial, J8 DUART I/O, J9 Free pin, SW1 HW_RESET_SW, U1 74LS05, U10 GAL22V10, U11 AS6C4008-55PCN, U12 AS6C4008-55PCN, U13 74LS245, U14 74LS245, U15 68681, U16 GAL22V10, U17 GAL22V10, U18 74LS244, U19 74LS244, U2 NE555P, U20 74LS175, U3 74LS244, U4 GAL22V10, U5 SST39SF040, U6 SST39SF040, U7 68010P10, U8 74LS244, U9 74LS244, X1 SG-8002DB 10Mhz

Commit message: updated readme
Parts:
- moved U18 21.4 mm to (452.1, 208.3)
Changed lines of the file:
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@@
   )
   (footprint "Package_DIP:DIP-20_W7.62mm_Socket" (layer "F.Cu")
-    (at 473.39 210.82)
+    (at 452.12 208.28)
     (descr "20-lead though-hole mounted DIP package, row spacing 7.62 mm (300 mils), Socket")
     (tags "THT DIP DIL PDIP 2.54mm 7.62mm 300mil Socket")
