File: kicad/_autosave-indicators.kicad_sch (KiCad schematic)
At the start: 36 parts, among them J9 Free pin, U14 74LS244

Commit message: saving state
Parts:
- C6: footprint Capacitor_THT:CP_Radial_D5.0mm_P2.50mm -> Capacitor_THT:C_Disc_D5.0mm_W2.5mm_P2.50mm
Changed lines of the file:
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@@
       (effects (font (size 1.27 1.27)) (justify left))
     )
-    (property "Footprint" "Capacitor_THT:CP_Radial_D5.0mm_P2.50mm" (at 119.0752 179.07 0)
+    (property "Footprint" "Capacitor_THT:C_Disc_D5.0mm_W2.5mm_P2.50mm" (at 119.0752 179.07 0)
       (effects (font (size 1.27 1.27)) hide)
     )
