File: kicad/_autosave-power.kicad_sch (KiCad schematic)
At the start: 17 parts, among them J25 ATX-24, J26 External Power, SW2 POWER ON

Commit message: saving state
Parts:
- added C2: 470uF, Capacitor_THT:CP_Radial_D5.0mm_P2.50mm, symbol Device:C_Polarized
- added C2: 100uF, Capacitor_THT:CP_Radial_D5.0mm_P2.50mm, symbol Device:C_Polarized
Connections:
- net GND: now also C2.2, C2.2
- net VCC: now also C2.1, C2.1
Changed lines of the file:
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@@
     (rev "1.0-alpha")
   )
+  (junction (at 236.22 69.85) (diameter 0) (color 0 0 0 0)
+  )
+  (junction (at 236.22 77.47) (diameter 0) (color 0 0 0 0)
+  )
   (junction (at 147.32 97.79) (diameter 0) (color 0 0 0 0)
+  )
+  (junction (at 251.46 69.85) (diameter 0) (color 0 0 0 0)
+  )
+  (junction (at 251.46 77.47) (diameter 0) (color 0 0 0 0)
   )
   (junction (at 184.15 77.47) (diameter 0) (color 0 0 0 0)
@@
     (stroke (width 0) (type default))
   )
+  (wire (pts (xy 251.46 77.47) (xy 264.16 77.47))
+    (stroke (width 0) (type default))
+  )
   (wire (pts (xy 120.65 69.85) (xy 120.65 97.79))
     (stroke (width 0) (type default))
   )
-  (wire (pts (xy 229.87 77.47) (xy 246.38 77.47))
+  (wire (pts (xy 229.87 77.47) (xy 236.22 77.47))
     (stroke (width 0) (type default))
   )
@@
     (stroke (width 0) (type default))
   )
+  (wire (pts (xy 236.22 77.47) (xy 251.46 77.47))
+    (stroke (width 0) (type default))
+  )
   (wire (pts (xy 229.87 39.37) (xy 229.87 77.47))
     (stroke (width 0) (type default))
@@
     (stroke (width 0) (type default))
   )
-  (wire (pts (xy 247.65 69.85) (xy 189.23 69.85))
+  (wire (pts (xy 236.22 69.85) (xy 189.23 69.85))
+    (stroke (width 0) (type default))
+  )
+  (wire (pts (xy 236.22 69.85) (xy 251.46 69.85))
     (stroke (width 0) (type default))
   )
@@
   )
   (wire (pts (xy 184.15 77.47) (xy 217.17 77.47))
+    (stroke (width 0) (type default))
+  )
+  (wire (pts (xy 251.46 69.85) (xy 264.16 69.85))
     (stroke (width 0) (type default))
   )
@@
     )
   )
-  (symbol (lib_id "power:GND") (at 247.65 69.85 90) (unit 1)
+  (symbol (lib_id "power:GND") (at 264.16 69.85 90) (unit 1)
     (in_bom yes) (on_board yes) (dnp no)
-    (property "Reference" "#PWR029" (at 254 69.85 0)
-      (effects (font (size 1.27 1.27)) hide)
-    )
-    (property "Value" "GND" (at 252.73 68.58 0)
-      (effects (font (size 1.27 1.27)) (justify right))
-    )
-    (property "Footprint" "" (at 247.65 69.85 0)
-      (effects (font (size 1.27 1.27)) hide)
-    )
-    (property "Datasheet" "" (at 247.65 69.85 0)
+    (property "Reference" "#PWR029" (at 270.51 69.85 0)
+      (effects (font (size 1.27 1.27)) hide)
+    )
+    (property "Value" "GND" (at 269.24 68.58 0)
+      (effects (font (size 1.27 1.27)) (justify right))
+    )
+    (property "Footprint" "" (at 264.16 69.85 0)
+      (effects (font (size 1.27 1.27)) hide)
+    )
+    (property "Datasheet" "" (at 264.16 69.85 0)
       (effects (font (size 1.27 1.27)) hide)
     )
@@
         (path "/e63e39d7-6ac0-4ffd-8aa3-1841a4541b55/917725a3-e126-410e-a107-b902da9d2a29"
           (reference "LED3") (unit 1)
+        )
+      )
+    )
+  )
+  (symbol (lib_id "Device:C_Polarized") (at 251.46 73.66 180) (unit 1)
+    (in_bom yes) (on_board yes) (dnp no) (fields_autoplaced)
+    (property "Reference" "C2" (at 255.27 73.279 0)
+      (effects (font (size 1.27 1.27)) (justify right))
+    )
+    (property "Value" "470uF" (at 255.27 75.819 0)
+      (effects (font (size 1.27 1.27)) (justify right))
+    )
+    (property "Footprint" "Capacitor_THT:CP_Radial_D5.0mm_P2.50mm" (at 250.4948 69.85 0)
+      (effects (font (size 1.27 1.27)) hide)
+    )
+    (property "Datasheet" "~" (at 251.46 73.66 0)
+      (effects (font (size 1.27 1.27)) hide)
+    )
+    (pin "1")
+    (pin "2")
+    (instances
+      (project "mb68k"
+        (path "/e63e39d7-6ac0-4ffd-8aa3-1841a4541b55/60b3e0cc-7d6f-4628-b20d-5a9d7b2fa5fa"
+          (reference "C2") (unit 1)
+        )
+        (path "/e63e39d7-6ac0-4ffd-8aa3-1841a4541b55/917725a3-e126-410e-a107-b902da9d2a29"
+          (reference "C17") (unit 1)
         )
       )
@@
     )
   )
-  (symbol (lib_id "power:VCC") (at 246.38 77.47 270) (unit 1)
-    (in_bom yes) (on_board yes) (dnp no) (fields_autoplaced)
-    (property "Reference" "#PWR028" (at 242.57 77.47 0)
-      (effects (font (size 1.27 1.27)) hide)
-    )
-    (property "Value" "VCC" (at 250.19 77.47 90)
-      (effects (font (size 1.27 1.27)) (justify left))
-    )
-    (property "Footprint" "" (at 246.38 77.47 0)
-      (effects (font (size 1.27 1.27)) hide)
-    )
-    (property "Datasheet" "" (at 246.38 77.47 0)
+  (symbol (lib_id "power:VCC") (at 264.16 77.47 270) (unit 1)
+    (in_bom yes) (on_board yes) (dnp no) (fields_autoplaced)
+    (property "Reference" "#PWR028" (at 260.35 77.47 0)
+      (effects (font (size 1.27 1.27)) hide)
+    )
+    (property "Value" "VCC" (at 267.97 77.47 90)
+      (effects (font (size 1.27 1.27)) (justify left))
+    )
+    (property "Footprint" "" (at 264.16 77.47 0)
+      (effects (font (size 1.27 1.27)) hide)
+    )
+    (property "Datasheet" "" (at 264.16 77.47 0)
       (effects (font (size 1.27 1.27)) hide)
     )
@@
         )
       )
+    )
+  )
+  (symbol (lib_id "Device:C_Polarized") (at 236.22 73.66 180) (unit 1)
+    (in_bom yes) (on_board yes) (dnp no) (fields_autoplaced)
+    (property "Reference" "C2" (at 240.03 73.279 0)
+      (effects (font (size 1.27 1.27)) (justify right))
+    )
+    (property "Value" "100uF" (at 240.03 75.819 0)
+      (effects (font (size 1.27 1.27)) (justify right))
+    )
+    (property "Footprint" "Capacitor_THT:CP_Radial_D5.0mm_P2.50mm" (at 235.2548 69.85 0)
+      (effects (font (size 1.27 1.27)) hide)
+    )
+    (property "Datasheet" "~" (at 236.22 73.66 0)
+      (effects (font (size 1.27 1.27)) hide)
+    )
+    (pin "1")
+    (pin "2")
+    (instances
+      (project "mb68k"
+        (path "/e63e39d7-6ac0-4ffd-8aa3-1841a4541b55/60b3e0cc-7d6f-4628-b20d-5a9d7b2fa5fa"
+          (reference "C2") (unit 1)
+        )
+        (path "/e63e39d7-6ac0-4ffd-8aa3-1841a4541b55/917725a3-e126-410e-a107-b902da9d2a29"
+          (reference "C16") (unit 1)
+        )
+      )
