File: kicad/busarb.kicad_sch (KiCad schematic)
At the start: 1 part, among them U13 74LS175

Commit message: switched to GALasm
Connections:
- net AS renamed _AS
Changed lines of the file:
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@@
     )
   )
-  (global_label "AS" (shape input) (at 36.83 97.79 180) (fields_autoplaced)
+  (global_label "_AS" (shape input) (at 36.83 97.79 180) (fields_autoplaced)
     (effects (font (size 1.27 1.27)) (justify right))
-    (property "Intersheetrefs" "${INTERSHEET_REFS}" (at 31.6261 97.79 0)
+    (property "Intersheetrefs" "${INTERSHEET_REFS}" (at 30.6585 97.79 0)
       (effects (font (size 1.27 1.27)) (justify right) hide)
     )

Commit message: added footprints
Parts:
- added C24: 100nF, Capacitor_THT:CP_Radial_D5.0mm_P2.50mm, symbol Device:C
- U20: renamed from U13; footprint (none) -> Package_DIP:DIP-16_W7.62mm_Socket
Connections:
- net GND: now also C24.1
- net VCC: now also C24.2
Changed lines of the file:
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@@
   (junction (at 43.18 97.79) (diameter 0) (color 0 0 0 0)
+  )
+  (junction (at 58.42 57.15) (diameter 0) (color 0 0 0 0)
+  )
+  (junction (at 58.42 106.68) (diameter 0) (color 0 0 0 0)
   )
   (no_connect (at 71.12 87.63))
@@
     (stroke (width 0) (type default))
   )
+  (wire (pts (xy 58.42 106.68) (xy 58.42 113.03))
+    (stroke (width 0) (type default))
+  )
+  (wire (pts (xy 82.55 83.82) (xy 82.55 106.68))
+    (stroke (width 0) (type default))
+  )
   (wire (pts (xy 38.1 85.09) (xy 45.72 85.09))
     (stroke (width 0) (type default))
@@
     (stroke (width 0) (type default))
   )
+  (wire (pts (xy 82.55 76.2) (xy 82.55 57.15))
+    (stroke (width 0) (type default))
+  )
   (wire (pts (xy 71.12 74.93) (xy 72.39 74.93))
     (stroke (width 0) (type default))
@@
     (stroke (width 0) (type default))
   )
-  (wire (pts (xy 58.42 105.41) (xy 58.42 113.03))
+  (wire (pts (xy 58.42 105.41) (xy 58.42 106.68))
     (stroke (width 0) (type default))
   )
@@
   )
   (wire (pts (xy 40.64 80.01) (xy 45.72 80.01))
+    (stroke (width 0) (type default))
+  )
+  (wire (pts (xy 82.55 57.15) (xy 58.42 57.15))
+    (stroke (width 0) (type default))
+  )
+  (wire (pts (xy 82.55 106.68) (xy 58.42 106.68))
     (stroke (width 0) (type default))
   )
@@
   (symbol (lib_id "power:VCC") (at 58.42 57.15 0) (unit 1)
     (in_bom yes) (on_board yes) (dnp no) (fields_autoplaced)
-    (property "Reference" "#PWR041" (at 58.42 60.96 0)
+    (property "Reference" "#PWR067" (at 58.42 60.96 0)
       (effects (font (size 1.27 1.27)) hide)
     )
@@
       (project "mb68k"
         (path "/e63e39d7-6ac0-4ffd-8aa3-1841a4541b55/9fd2bd3c-9347-4575-b465-a62477559a86"
-          (reference "#PWR041") (unit 1)
+          (reference "#PWR067") (unit 1)
+        )
+      )
+    )
+  )
+  (symbol (lib_id "Device:C") (at 82.55 80.01 0) (mirror x) (unit 1)
+    (in_bom yes) (on_board yes) (dnp no)
+    (property "Reference" "C24" (at 90.17 80.01 90)
+      (effects (font (size 1.27 1.27)))
+    )
+    (property "Value" "100nF" (at 87.63 80.01 90)
+      (effects (font (size 1.27 1.27)))
+    )
+    (property "Footprint" "Capacitor_THT:CP_Radial_D5.0mm_P2.50mm" (at 83.5152 76.2 0)
+      (effects (font (size 1.27 1.27)) hide)
+    )
+    (property "Datasheet" "~" (at 82.55 80.01 0)
+      (effects (font (size 1.27 1.27)) hide)
+    )
+    (pin "1")
+    (pin "2")
+    (instances
+      (project "mb68k"
+        (path "/e63e39d7-6ac0-4ffd-8aa3-1841a4541b55/6c955f8d-27cd-4aef-8df3-4a7f3323692c"
+          (reference "C24") (unit 1)
+        )
+        (path "/e63e39d7-6ac0-4ffd-8aa3-1841a4541b55/9fd2bd3c-9347-4575-b465-a62477559a86"
+          (reference "C26") (unit 1)
         )
       )
@@
   (symbol (lib_id "power:GND") (at 58.42 113.03 0) (unit 1)
     (in_bom yes) (on_board yes) (dnp no) (fields_autoplaced)
-    (property "Reference" "#PWR040" (at 58.42 119.38 0)
+    (property "Reference" "#PWR068" (at 58.42 119.38 0)
       (effects (font (size 1.27 1.27)) hide)
     )
@@
       (project "mb68k"
         (path "/e63e39d7-6ac0-4ffd-8aa3-1841a4541b55/9fd2bd3c-9347-4575-b465-a62477559a86"
-          (reference "#PWR040") (unit 1)
+          (reference "#PWR068") (unit 1)
         )
       )
@@
   (symbol (lib_id "74xx:74LS175") (at 58.42 85.09 0) (unit 1)
     (in_bom yes) (on_board yes) (dnp no) (fields_autoplaced)
-    (property "Reference" "U13" (at 60.3759 67.31 0)
+    (property "Reference" "U20" (at 60.3759 67.31 0)
       (effects (font (size 1.27 1.27)) (justify left))
     )
@@
       (effects (font (size 1.27 1.27)) (justify left))
     )
-    (property "Footprint" "" (at 58.42 85.09 0)
+    (property "Footprint" "Package_DIP:DIP-16_W7.62mm_Socket" (at 58.42 85.09 0)
       (effects (font (size 1.27 1.27)) hide)
     )
@@
       (project "mb68k"
         (path "/e63e39d7-6ac0-4ffd-8aa3-1841a4541b55/9fd2bd3c-9347-4575-b465-a62477559a86"
-          (reference "U13") (unit 1)
-        )
-      )
+          (reference "U20") (unit 1)
+        )
+      )

Commit message: saving state
Parts:
- C24: footprint Capacitor_THT:CP_Radial_D5.0mm_P2.50mm -> Capacitor_THT:C_Disc_D5.0mm_W2.5mm_P2.50mm
Changed lines of the file:
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@@
       (effects (font (size 1.27 1.27)))
     )
-    (property "Footprint" "Capacitor_THT:CP_Radial_D5.0mm_P2.50mm" (at 83.5152 76.2 0)
+    (property "Footprint" "Capacitor_THT:C_Disc_D5.0mm_W2.5mm_P2.50mm" (at 83.5152 76.2 0)
       (effects (font (size 1.27 1.27)) hide)
     )
