File: kicad/indicators.kicad_sch (KiCad schematic)
At the start: 36 parts, among them J9 Free pin, U14 74LS244

Commit message: saving kicad
Connections:
- net ~{IRQ5}: now also U14.15 (I2b); no longer U14.11 (I0b)
- net ~{IRQ7}: now also U14.11 (I0b); no longer U14.15 (I2b)
Changed lines of the file:
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@@
     )
   )
-  (global_label "~{IRQ5}" (shape input) (at 85.09 45.72 180) (fields_autoplaced)
+  (global_label "~{IRQ5}" (shape input) (at 85.09 50.8 180) (fields_autoplaced)
     (effects (font (size 1.27 1.27)) (justify right))
-    (property "Intersheetrefs" "${INTERSHEET_REFS}" (at 77.7694 45.72 0)
+    (property "Intersheetrefs" "${INTERSHEET_REFS}" (at 77.7694 50.8 0)
       (effects (font (size 1.27 1.27)) (justify right) hide)
     )
@@
     )
   )
-  (global_label "~{IRQ7}" (shape input) (at 85.09 50.8 180) (fields_autoplaced)
+  (global_label "~{IRQ7}" (shape input) (at 85.09 45.72 180) (fields_autoplaced)
     (effects (font (size 1.27 1.27)) (justify right))
-    (property "Intersheetrefs" "${INTERSHEET_REFS}" (at 77.7694 50.8 0)
+    (property "Intersheetrefs" "${INTERSHEET_REFS}" (at 77.7694 45.72 0)
       (effects (font (size 1.27 1.27)) (justify right) hide)
     )

Commit message: fiddlign with placement
Connections:
- net at U14.5 (O2b): now also D3.1 (K); no longer D1.1 (K)
- net at U14.9 (O0b): now also D1.1 (K); no longer D3.1 (K)
Changed lines of the file:
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@@
+    (stroke (width 0) (type default))
+  )
+  (wire (pts (xy 191.77 45.72) (xy 135.89 45.72))
     (stroke (width 0) (type default))
   )
@@
     (stroke (width 0) (type default))
   )
+  (wire (pts (xy 135.89 45.72) (xy 135.89 50.8))
+    (stroke (width 0) (type default))
+  )
   (wire (pts (xy 87.63 127) (xy 87.63 129.54))
     (stroke (width 0) (type default))
@@
     (stroke (width 0) (type default))
   )
+  (wire (pts (xy 121.92 45.72) (xy 114.3 45.72))
+    (stroke (width 0) (type default))
+  )
   (wire (pts (xy 85.09 104.14) (xy 88.9 104.14))
     (stroke (width 0) (type default))
   )
+  (wire (pts (xy 135.89 50.8) (xy 114.3 50.8))
+    (stroke (width 0) (type default))
+  )
   (wire (pts (xy 101.6 72.39) (xy 101.6 74.93))
     (stroke (width 0) (type default))
@@
     (stroke (width 0) (type default))
   )
-  (wire (pts (xy 114.3 45.72) (xy 191.77 45.72))
-    (stroke (width 0) (type default))
-  )
-  (wire (pts (xy 114.3 50.8) (xy 189.23 50.8))
-    (stroke (width 0) (type default))
-  )
   (wire (pts (xy 243.84 80.01) (xy 243.84 71.12))
     (stroke (width 0) (type default))
@@
     (stroke (width 0) (type default))
   )
-  (wire (pts (xy 189.23 50.8) (xy 189.23 88.9))
+  (wire (pts (xy 189.23 46.99) (xy 189.23 88.9))
     (stroke (width 0) (type default))
   )
@@
     (stroke (width 0) (type default))
   )
+  (wire (pts (xy 189.23 46.99) (xy 121.92 46.99))
+    (stroke (width 0) (type default))
+  )
   (wire (pts (xy 114.3 106.68) (xy 193.04 106.68))
     (stroke (width 0) (type default))
@@
     (stroke (width 0) (type default))
   )
+  (wire (pts (xy 121.92 46.99) (xy 121.92 45.72))
+    (stroke (width 0) (type default))
+  )

Commit message: got irq to work
Parts:
- removed R18 (x3), R19 (x3), R20 (x8): R330, Resistor_THT:R_Axial_DIN0207_L6.3mm_D2.5mm_P10.16mm_Horizontal, symbol Device:R
- added RN1 (x2): R_Network08, Resistor_THT:R_Array_SIP9, symbol Device:R_Network08
Connections:
- net GND: now also RN1.1 (common)
- net VCC: now also RN1.1 (common)
- net at D3.2 (A): now also RN1.3 (R2)
- net at D1.1 (K): now also RN1.5 (R4)
- net at D2.2 (A): now also RN1.5 (R4)
- net at D2.2 (A): now also RN1.2 (R1)
- net at D3.1 (K): now also RN1.3 (R2)
- net at D1.1 (K): now also RN1.4 (R3)
- net at D1.1 (K): now also RN1.8 (R7)
- net at D1.1 (K): now also RN1.6 (R5)
- net at D1.2 (A): now also RN1.4 (R3)
- net at D1.2 (A): now also RN1.7 (R6)
- net at D2.1 (K): now also RN1.2 (R1)
- net at D1.1 (K): now also RN1.7 (R6)
- net at D1.2 (A): now also RN1.8 (R7)
- net at D3.2 (A): now also RN1.6 (R5)
- no-connect marks 0 -> 2
